File: board/kicad/tonnere/audio.kicad_sch (KiCad schematic)
At the start: 40 parts, among them J1 PJ-325C5-G, J2 PJ-325C5-BL, U19 PCM5102A

Commit message: Made audio connector stacked. Added S/PDIF toslink output
Parts:
- removed J1: PJ-325C5-G, Connector_Audio:Jack_3.5mm_CUI_SJ1-3535NG_Horizontal, symbol Connector_Audio:AudioJack3_SwitchTR
- removed J2: PJ-325C5-BL, Connector_Audio:Jack_3.5mm_CUI_SJ1-3535NG_Horizontal, symbol Connector_Audio:AudioJack3_SwitchTR
- added C126: 0.1uF, Capacitor_SMD:C_0603_1608Metric, symbol Device:C
- added J28: JA23331-HA6Q-4F, tonnere:AUDIO-TH_JA23331-HA6Q-4F, symbol tonnere:JA23331-HA6Q-4F
- added U48: PLT237/T10WH, tonnere:CONN-TH_PLT237-T10WH, symbol tonnere:PLT237_T10WH
Connections:
- net GND: now also C126.1, U48.3 (GND)
- net GNDA: now also J28.1, J28.6 (EH), J28.7 (EH), J28.8 (EH), J28.9 (EH)
- net at C3.2, R6.2: now also J28.25
- net at C2.2, R2.2: now also J28.22
- net at C1.2, R1.2: now also J28.2
- net at C4.2, R8.2: now also J28.5
- new net +5V: C126.2, U48.1 (Vin)
- new net FPGAAUD.SPDIF: U48.2 (VCC)
