File: board/kicad/tonnere/audio.kicad_sch (KiCad schematic)
At the start: 41 parts, among them J28 JA23331-HA6Q-4F, U19 PCM5102A, U48 PLT237/T10WH

Commit message: Changed video dac to 5 bit R2R and 6th-8th bits as pattern and/or sigma delta.
Parts:
- C30: renamed from C29; value 4.7nF -> 10nF; LCSC C53987 -> C57112
- C34: renamed from C33; value 4.7nF -> 10nF; LCSC C53987 -> C57112
- C48: renamed from C46; value 4.7nF -> 10nF; LCSC C53987 -> C57112
- C52: renamed from C51; value 4.7nF -> 10nF; LCSC C53987 -> C57112
- renumbered C9 to C10, C102 to C103, C103 to C104, C23 to C24, C26 to C27, C27 to C28, C126 to C3, C39 to C40, C48 to C47, C47 to C49, C4 to C5, C3 to C6, C6 to C7, C8 to C9, J28 to J4, R115 to R110, R116 to R111, R8 to R18, R20 to R19, R10 to R20, R48 to R51, R56 to R59, R59 to R62, U48 to U1, U19 to U20
Connections:
- net GND: no longer C10.1, C30.1, C34.1, C48.1, C52.1, C9.1, R29.2
- net GNDA: now also C10.1, C30.1, C34.1, C48.1, C52.1, C9.1, R29.2
- net Net-(U19-LDOO): now reaches C40.2, U20.18 (LDOO)
- net Net-(C102-Pad2): now reaches C103.2, C104.2, R25.1, R62.2
- net Net-(C4-Pad1): now reaches C5.1, R19.1, R43.2
- net unconnected-(U48-NC-Pad4): now reaches U1.4 (NC)
- net unconnected-(U48-NC-Pad5): now reaches U1.5 (NC)
- net Net-(C3-Pad2): now reaches C6.2, J4.25, R6.2
- net unconnected-(J28-Pad23): now reaches J4.23
- net unconnected-(J28-Pad24): now reaches J4.24
- net unconnected-(J28-Pad3): now reaches J4.3
- net unconnected-(J28-Pad4): now reaches J4.4
- net Net-(C4-Pad2): now reaches C5.2, J4.5, R18.2
- net Net-(C8-Pad2): now reaches C10.2, C9.2, R19.2, R20.2, R25.2, R26.2, R27.2, R29.1
- net Net-(C6-Pad2): now reaches C7.2, R26.1, R59.2
- net Net-(C103-Pad1): now reaches C104.1, R110.2
- net Net-(U19-CAPP): now reaches C28.2, U20.2 (CAPP)
- net Net-(U19-CAPM): now reaches C28.1, U20.4 (CAPM)
- net Net-(U19-VNEG): now reaches C24.2, U20.5 (VNEG)
- net Net-(U19-OUTL): now reaches R2.1, U20.6 (OUTL)
- net Net-(U19-OUTR): now reaches R6.1, U20.7 (OUTR)
- no-connect marks 4 -> 6
