File: board/kicad/tonnere/cycloneve.kicad_sch (KiCad schematic)
At the start: 54 parts, among them J15 SPI CFG, J17 SPI SEL, J22 FPGA JTAG, U27 M25PX32-VMW, U29 M25PX32-VMW, U33 10CL040f484, Y4 25MHz, Y5 Si5351A-B-GT, Y6 ASE-27MHz, Y7 25MHz, Y8 Si5351A-B-GT

Commit message: Made audio connector stacked. Added S/PDIF toslink output
Connections:
- net FPGAAUD.SPDIF: now reaches U33.G4 (DIFFIO_L1p)
- no-connect marks 35 -> 34
Changed lines of the file:
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@@
 	)
 	(no_connect
-		(at 111.76 96.52)
-	)
-	(no_connect
 		(at 581.66 96.52)
 	)
@@
 	)
 	(bus_entry
+		(at 72.39 91.44)
+		(size 2.54 2.54)
+		(stroke
+			(width 0)
+			(type default)
+		)
+	)
+	(bus_entry
 		(at 335.28 71.12)
 		(size 2.54 2.54)
@@
 		)
 	)
+	(bus
+		(pts
+			(xy 72.39 91.44) (xy 72.39 92.71)
+		)
+		(stroke
+			(width 0)
+			(type default)
+		)
+	)
 	(wire
 		(pts
@@
 		)
 	)
+	(wire
+		(pts
+			(xy 77.47 95.25) (xy 90.17 95.25)
+		)
+		(stroke
+			(width 0)
+			(type default)
+		)
+	)
 	(bus
 		(pts
@@
 	(wire
 		(pts
+			(xy 77.47 93.98) (xy 77.47 95.25)
+		)
+		(stroke
+			(width 0)
+			(type default)
+		)
+	)
+	(wire
+		(pts
 			(xy 427.99 213.36) (xy 444.5 213.36)
 		)
@@
 	(wire
 		(pts
+			(xy 74.93 93.98) (xy 77.47 93.98)
+		)
+		(stroke
+			(width 0)
+			(type default)
+		)
+	)
+	(wire
+		(pts
 			(xy 255.27 405.13) (xy 250.19 405.13)
 		)
@@
 	(wire
 		(pts
+			(xy 90.17 96.52) (xy 111.76 96.52)
+		)
+		(stroke
+			(width 0)
+			(type default)
+		)
+	)
+	(wire
+		(pts
 			(xy 469.9 254) (xy 485.14 254)
 		)
@@
 	(wire
 		(pts
+			(xy 90.17 95.25) (xy 90.17 96.52)
+		)
+		(stroke
+			(width 0)
+			(type default)
+		)
+	)
+	(wire
+		(pts
 			(xy 361.95 421.64) (xy 361.95 426.72)
 		)
@@
 	(bus
 		(pts
-			(xy 72.39 76.2) (xy 72.39 92.71)
+			(xy 72.39 76.2) (xy 72.39 91.44)
 		)
 		(stroke
@@
 		)
 	)
+	(label "FPGAAUD.SPDIF"
+		(at 92.71 96.52 0)
+		(effects
+			(font
+				(size 1.27 1.27)
+			)
+			(justify left bottom)
+		)
+	)
 	(label "FSMC.A2"
 		(at 570.23 257.81 0)
@@
 		)
 	)
-	(hierarchical_label "FPGAAUD{DATA,BCK,LR}"
+	(hierarchical_label "FPGAAUD{DATA,BCK,LR,SPDIF}"
 		(shape bidirectional)
 		(at 64.77 92.71 180)
