File: board/kicad/tonnere/cycloneve.kicad_sch (KiCad schematic)
At the start: 54 parts, among them J15 SPI CFG, J17 SPI SEL, J22 FPGA JTAG, U27 M25PX32-VMW, U29 M25PX32-VMW, U33 10CL040f484, Y4 25MHz, Y5 Si5351A-B-GT, Y6 ASE-27MHz, Y7 25MHz, Y8 Si5351A-B-GT

Commit message: Changed video dac to 5 bit R2R and 6th-8th bits as pattern and/or sigma delta.
Parts:
- renumbered C99 to C100, C101 to C102, C113 to C114, C116 to C117, C65 to C69, C70 to C71, C72 to C73, C75 to C74, C74 to C75, C73 to C82, C83 to C87, C88 to C89, C90 to C91, C91 to C92, C96 to C97, FB5 to FB4, FB7 to FB6, J15 to J14, J17 to J16, J22 to J21, R118 to R113, R120 to R115, R123 to R118, R126 to R121, R129 to R124, R130 to R125, R131 to R126, R74 to R77, R69 to R78, R70 to R79, R71 to R80, R75 to R82, R76 to R83, R84 to R86, R92 to R87, R93 to R88, R95 to R90, R96 to R91, R97 to R92, R99 to R94, R101 to R96, R102 to R97, R104 to R99, U27 to U28, U29 to U30, U33 to U34
Connections:
- net unconnected-(U33A-DIFFIO_L14n-PadJ8) is gone; now on net FPGA.GPIO1: U34.J8 (DIFFIO_L14n)
- net unconnected-(U33A-DIFFIO_L14p-PadH8) is gone; now on net FPGA.GPIO2: U34.H8 (DIFFIO_L14p)
- net unconnected-(U33A-DIFFIO_L20n-PadK8) is gone; now on net FPGA.GPIO3: U34.K8 (DIFFIO_L20n)
- net unconnected-(U33A-DIFFIO_L20p-PadL8) is gone; now on net FPGA.GPIO4: U34.L8 (DIFFIO_L20p)
- net unconnected-(U33A-DIFFIO_L2n-PadB1) is gone; now on net VDAC.B0: U34.B1 (DIFFIO_L2n)
- net unconnected-(U33A-DIFFIO_L2p-PadB2) is gone; now on net VDAC.B1: U34.B2 (DIFFIO_L2p)
- net unconnected-(U33A-IO-PadH7) is gone; now on net FPGAAUD.SPDIF: U34.H7 (IO)
- net unconnected-(U33H-IO-PadG7) is gone; now on net FPGA.GPIO0: U34.G7 (IO)
- net FPGA.GPIO0: no longer U34.C3 (IO)
- net FPGA.GPIO1: no longer U34.B3 (IO)
- net FPGA.GPIO2: no longer U34.C4 (IO)
- net FPGA.GPIO3: no longer U34.B4 (IO)
- net FPGA.GPIO4: no longer U34.A4 (IO)
- net FPGAAUD.BCK: now also U34.B3 (IO); no longer U34.D2 (DIFFIO_L8p)
- net FPGAAUD.DATA: now also U34.B4 (IO); no longer U34.J4 (IO)
- net FPGAAUD.LR: now also U34.A4 (IO); no longer U34.G5 (IO)
- net FPGAAUD.SPDIF: no longer U34.G4 (DIFFIO_L1p)
- net VDAC.B0: no longer U34.H1 (DIFFIO_L23n)
- net VDAC.B1: no longer U34.H2 (DIFFIO_L23p)
- net VDAC.B2: now also U34.C3 (IO); no longer U34.J3 (IO)
- net VDAC.G0: now also U34.E1 (DIFFIO_L10n); no longer U34.F1 (DIFFIO_L12n)
- net VDAC.G1: now also U34.E3 (DIFFIO_L4n); no longer U34.F2 (DIFFIO_L12p)
- net VDAC.G2: now also U34.G4 (DIFFIO_L1p); no longer U34.G3 (DIFFIO_L1n)
- net VDAC.R0: now also U34.G3 (DIFFIO_L1n); no longer U34.E1 (DIFFIO_L10n)
- net VDAC.R1: now also U34.F2 (DIFFIO_L12p); no longer U34.E3 (DIFFIO_L4n)
- net VDAC.R2: now also U34.F1 (DIFFIO_L12n); no longer U34.E4 (DIFFIO_L4p)
- net unconnected-(J22-Pin_6-Pad6): now reaches J21.6 (Pin_6)
- net unconnected-(J22-Pin_7-Pad7): now reaches J21.7 (Pin_7)
- net unconnected-(J22-Pin_8-Pad8): now reaches J21.8 (Pin_8)
- net Net-(U27-DQ1): now reaches R80.1, U28.2 (DQ1)
- net Net-(J17-Pin_3): now reaches J16.3 (Pin_3), R82.2, U28.1 (~{S})
- net Net-(J17-Pin_1): now reaches J16.1 (Pin_1), R94.2, U30.1 (~{S}/~{CS})
- net Net-(U29-DQ1/SO): now reaches R91.1, U30.2 (DQ1/SO)
- net Net-(U27-~{W}/V_{PP}): now reaches R78.2, U28.3 (~{W}/V_{PP}), U30.3 (~{W}/V_{PP})
- net Net-(U27-~{HOLD}): now reaches R79.2, U28.7 (~{HOLD}), U30.7 (~{HOLD})
- net unconnected-(U33A-DIFFIO_L21n-PadK7) renamed unconnected-(U33bank1-DIFFIO_L21n-PadK7)
- net unconnected-(U33A-DIFFIO_L9p-PadH6) renamed VDAC.G4
- net unconnected-(U33A-IO-PadH5) renamed VDAC.G5
- new net VDAC.B3: U34.C4 (IO)
- new net VDAC.B4: U34.D2 (DIFFIO_L8p)
- new net VDAC.B5: U34.E4 (DIFFIO_L4p)
- new net VDAC.G3: U34.G5 (IO)
- new net VDAC.R3: U34.J3 (IO)
- new net VDAC.R4: U34.H2 (DIFFIO_L23p)
- new net VDAC.R5: U34.H1 (DIFFIO_L23n)
- new net unconnected-(U33bank1-IO-PadJ4): U34.J4 (IO)
- no-connect marks 34 -> 25
