File: board/kicad/tonnere/tonnere.kicad_sch (KiCad schematic)
At the start: 10 parts

Commit message: Made audio connector stacked. Added S/PDIF toslink output
Other:
- sheet Audio ports: added FPGAAUD{DATA,BCK,LR,SPDIF}; removed FPGAAUD{DATA,BCK,LR}
- sheet FPGA ports: added FPGAAUD{DATA,BCK,LR,SPDIF}; removed FPGAAUD{DATA,BCK,LR}
Changed lines of the file:
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@@
 			)
 		)
-		(pin "FPGAAUD{DATA,BCK,LR}" bidirectional
+		(pin "FPGAAUD{DATA,BCK,LR,SPDIF}" bidirectional
 			(at 229.87 107.95 180)
 			(effects
@@
 			)
 		)
-		(pin "FPGAAUD{DATA,BCK,LR}" bidirectional
-			(at 29.21 59.69 90)
-			(effects
-				(font
-					(size 1.27 1.27)
-				)
-				(justify right)
-			)
-		)
 		(pin "JOY2{DIR[8..15],TRIG[2..3],POT[4..7]}" bidirectional
 			(at 119.38 90.17 0)
@@
 			(effects
 				(font
+					(size 1.27 1.27)
+				)
+				(justify right)
+			)
+		)
+		(pin "FPGAAUD{DATA,BCK,LR,SPDIF}" bidirectional
+			(at 29.21 59.69 90)
+			(effects
+				(font
