File: board/kicad/tonnere/tonnere.kicad_sch (KiCad schematic)
At the start: 10 parts

Commit message: Changed video dac to 5 bit R2R and 6th-8th bits as pattern and/or sigma delta.
Other:
- sheet FPGA ports: added VDAC{R[0..5],G[0..5],B[0..5],HSYNC,VSYNC}; removed VDAC{R[0..2],G[0..2],B[0..2],HSYNC,VSYNC}
- sheet Video ports: added VDAC{R[0..5],G[0..5],B[0..5],HSYNC,VSYNC}; removed VDAC{R[0..2],G[0..2],B[0..2],HSYNC,VSYNC}
Changed lines of the file:
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@@
 			)
 		)
-		(pin "VDAC{R[0..2],G[0..2],B[0..2],HSYNC,VSYNC}" bidirectional
+		(pin "VDAC{R[0..5],G[0..5],B[0..5],HSYNC,VSYNC}" bidirectional
 			(at 134.62 152.4 180)
 			(effects
@@
 			)
 		)
-		(pin "VDAC{R[0..2],G[0..2],B[0..2],HSYNC,VSYNC}" bidirectional
-			(at 119.38 85.09 0)
-			(effects
-				(font
-					(size 1.27 1.27)
-				)
-				(justify right)
-			)
-		)
 		(pin "FPGAAUD{DATA,BCK,LR,SPDIF}" bidirectional
 			(at 29.21 59.69 90)
 			(effects
 				(font
+					(size 1.27 1.27)
+				)
+				(justify right)
+			)
+		)
+		(pin "VDAC{R[0..5],G[0..5],B[0..5],HSYNC,VSYNC}" bidirectional
+			(at 119.38 85.09 0)
+			(effects
+				(font
