File: board/kicad/tonnere/atariinterfaces.kicad_sch (KiCad schematic)
At the start: 70 parts, among them J18 FPGA GPIO, J24 CONSOL, J6 PBI, J7 Conn_01x01, J8 PBI Option, Q1 BCX51, U10 TPD8E003DQDR, U13 TPD8E003DQDR, U14 TPD8E003DQDR, U18 TPD8E003DQDR, U24 TPD8E003DQDR, U28 TPD8E003DQDR, U30 SN74CB3T16211DGVR, U32 SN74CB3T16211DGVR, U35 SN74CB3T16211DGVR, U37 SN74CB3T16211DGVR, U5 TPD8E003DQDR, U6 TPD8E003DQDR, U7 TPD8E003DQDR, U8 TPD8E003DQDR, U9 TPD8E003DQDR

Commit message: Changed video dac to 5 bit R2R and 6th-8th bits as pattern and/or sigma delta.
Parts:
- renumbered C11 to C12, C13 to C14, C38 to C39, C5 to C4, C43 to C44, C56 to C60, C58 to C64, C71 to C72, C92 to C93, C97 to C98, J3 to J1, J11 to J10, J13 to J12, J16 to J15, J18 to J17, J24 to J23, J6 to J5, J7 to J6, J8 to J7, R12 to R10, R13 to R11, R15 to R13, R49 to R52, R50 to R53, R58 to R61, R67 to R70, R68 to R72, R72 to R81, R94 to R89, R11 to R9, R98 to R93, R100 to R95, RN11 to RN19, U9 to U10, U10 to U11, U13 to U14, U14 to U15, U18 to U19, U24 to U26, U28 to U29, U30 to U31, U32 to U33, U35 to U36, U37 to U38, U5 to U6, U6 to U7, U7 to U8, U8 to U9
Connections:
- net Net-(J16A-POTA): now reaches J15.9 (POTA), R89.2
- net Net-(J16B-POTA): now reaches J15.18 (POTA), R70.2
- net Net-(J11A-POTB): now reaches J10.5 (POTB), R53.2
- net unconnected-(U13-IO1-Pad1): now reaches U14.1 (IO1)
- net unconnected-(U13-IO2-Pad2): now reaches U14.2 (IO2)
- net unconnected-(U13-IO3-Pad3): now reaches U14.3 (IO3)
- net unconnected-(U13-IO4-Pad4): now reaches U14.4 (IO4)
- net unconnected-(U13-IO6-Pad6): now reaches U14.6 (IO6)
- net unconnected-(U13-IO7-Pad7): now reaches U14.7 (IO7)
- net Net-(J16B-POTB): now reaches J15.14 (POTB), R72.2
- net Net-(J11A-POTA): now reaches J10.9 (POTA), R52.2
- net Net-(J16A-POTB): now reaches J15.5 (POTB), R93.2
- net Net-(J11B-POTB): now reaches J10.14 (POTB), R36.2
- net Net-(J11B-POTA): now reaches J10.18 (POTA), R30.2
- net unconnected-(U35-NC-Pad1): now reaches U36.1 (NC)
- net unconnected-(U35-2A6-Pad22): now reaches U36.22 (2A6)
- net unconnected-(U35-2A7-Pad23): now reaches U36.23 (2A7)
- net unconnected-(U35-2A8-Pad24): now reaches U36.24 (2A8)
- net unconnected-(U35-2A9-Pad25): now reaches U36.25 (2A9)
- net unconnected-(U35-2A10-Pad26): now reaches U36.26 (2A10)
- net unconnected-(U35-2A11-Pad27): now reaches U36.27 (2A11)
- net unconnected-(U35-2A12-Pad28): now reaches U36.28 (2A12)
- net unconnected-(U35-2B12-Pad29): now reaches U36.29 (2B12)
- net unconnected-(U35-2B11-Pad30): now reaches U36.30 (2B11)
- net unconnected-(U35-2B10-Pad31): now reaches U36.31 (2B10)
- net unconnected-(U35-2B9-Pad32): now reaches U36.32 (2B9)
- net unconnected-(U35-2B8-Pad33): now reaches U36.33 (2B8)
- net unconnected-(U35-2B7-Pad34): now reaches U36.34 (2B7)
- net unconnected-(U35-2B6-Pad35): now reaches U36.35 (2B6)
- net unconnected-(U18-IO1-Pad1): now reaches U19.1 (IO1)
- net unconnected-(U30-NC-Pad1): now reaches U31.1 (NC)
- net unconnected-(U37-NC-Pad1): now reaches U38.1 (NC)
- net unconnected-(U32-NC-Pad1): now reaches U33.1 (NC)
- net unconnected-(U32-1B6-Pad48): now reaches U33.48 (1B6)
- net Net-(J18-Pin_7): now reaches J17.7 (Pin_7), U33.50 (1B5)
- net Net-(J18-Pin_6): now reaches J17.6 (Pin_6), U33.51 (1B4)
- net Net-(J18-Pin_5): now reaches J17.5 (Pin_5), U33.52 (1B3)
- net Net-(J18-Pin_4): now reaches J17.4 (Pin_4), U33.53 (1B2)
- net Net-(J18-Pin_3): now reaches J17.3 (Pin_3), U33.54 (1B1)
- net unconnected-(U32-1A6-Pad7): now reaches U33.7 (1A6)
- net unconnected-(U14-IO1-Pad1): now reaches U15.1 (IO1)
- net unconnected-(J3-+12V-Pad12): now reaches J1.12 (+12V)
- net unconnected-(U24-IO1-Pad1): now reaches U26.1 (IO1)
- net unconnected-(U28-IO1-Pad1): now reaches U29.1 (IO1)
