File: board/kicad/tonnere/esp32.kicad_sch (KiCad schematic)
At the start: 11 parts, among them J19 ESP PGM, J23 ESP JTAG, U40 ESP32-WROVER-E-N8R8

Commit message: Changed video dac to 5 bit R2R and 6th-8th bits as pattern and/or sigma delta.
Parts:
- renumbered C115 to C116, C117 to C118, J19 to J18, J23 to J22, R106 to R101, R108 to R103, R110 to R105, R113 to R108, R121 to R116, R103 to R98, U40 to U41
Connections:
- net unconnected-(J23-Pin_6-Pad6): now reaches J22.6 (Pin_6)
- net unconnected-(J23-Pin_7-Pad7): now reaches J22.7 (Pin_7)
- net unconnected-(J23-Pin_8-Pad8): now reaches J22.8 (Pin_8)
- net unconnected-(U40-NC-Pad17): now reaches U41.17 (NC)
- net unconnected-(U40-NC-Pad18): now reaches U41.18 (NC)
- net unconnected-(U40-NC-Pad19): now reaches U41.19 (NC)
- net unconnected-(U40-NC-Pad20): now reaches U41.20 (NC)
- net unconnected-(U40-NC-Pad21): now reaches U41.21 (NC)
- net unconnected-(U40-NC-Pad22): now reaches U41.22 (NC)
- net unconnected-(U40-NC-Pad27): now reaches U41.27 (NC)
- net unconnected-(U40-NC-Pad28): now reaches U41.28 (NC)
- net unconnected-(U40-NC-Pad32): now reaches U41.32 (NC)
Changed lines of the file:
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@@
+		)
+	)
+	(label "unconnected-(U40-NC-Pad19)"
+		(at 119.38 153.67 180)
+		(effects
+			(font
+				(size 1.27 1.27)
+			)
+			(justify right bottom)
 		)
 	)
@@
 		)
 	)
+	(label "unconnected-(U40-NC-Pad22)"
+		(at 149.86 148.59 0)
+		(effects
+			(font
+				(size 1.27 1.27)
+			)
+			(justify left bottom)
+		)
+	)
+	(label "unconnected-(U40-NC-Pad17)"
+		(at 119.38 148.59 180)
+		(effects
+			(font
+				(size 1.27 1.27)
+			)
+			(justify right bottom)
+		)
+	)
 	(label "ESPJTAG{TMS,TCK,TDI,TDO}"
 		(at 36.83 147.32 0)
@@
 		)
 	)
+	(label "unconnected-(J23-Pin_7-Pad7)"
+		(at 44.45 165.1 180)
+		(effects
+			(font
+				(size 1.27 1.27)
+			)
+			(justify right bottom)
+		)
+	)
 	(label "SIO.CLOCK_IN"
 		(at 153.67 120.65 0)
@@
 		)
 	)
+	(label "unconnected-(J23-Pin_6-Pad6)"
+		(at 57.15 162.56 0)
+		(effects
+			(font
+				(size 1.27 1.27)
+			)
+			(justify left bottom)
+		)
+	)
 	(label "ESP.SGPI0"
 		(at 100.33 115.57 0)
@@
 		)
 	)
+	(label "unconnected-(U40-NC-Pad32)"
+		(at 149.86 123.19 0)
+		(effects
+			(font
+				(size 1.27 1.27)
+			)
+			(justify left bottom)
+		)
+	)
 	(label "ESPJTAG.TDI"
 		(at 87.63 140.97 0)
@@
 		)
 	)
+	(label "unconnected-(U40-NC-Pad21)"
+		(at 149.86 151.13 0)
+		(effects
+			(font
+				(size 1.27 1.27)
+			)
+			(justify left bottom)
+		)
+	)
 	(label "ESP.MISO"
 		(at 162.56 125.73 0)
@@
 		)
 	)
+	(label "unconnected-(U40-NC-Pad27)"
+		(at 149.86 135.89 0)
+		(effects
+			(font
+				(size 1.27 1.27)
+			)
+			(justify left bottom)
+		)
+	)
 	(label "UART1.RX"
 		(at 218.44 115.57 0)
@@
 		)
 	)
+	(label "unconnected-(U40-NC-Pad20)"
+		(at 149.86 153.67 0)
+		(effects
+			(font
+				(size 1.27 1.27)
+			)
+			(justify left bottom)
+		)
+	)
+	(label "unconnected-(U40-NC-Pad18)"
+		(at 119.38 151.13 180)
+		(effects
+			(font
+				(size 1.27 1.27)
+			)
+			(justify right bottom)
+		)
+	)
 	(label "ESP.MOSI"
 		(at 162.56 110.49 0)
@@
 		)
 	)
+	(label "unconnected-(J23-Pin_8-Pad8)"
+		(at 57.15 165.1 0)
+		(effects
+			(font
+				(size 1.27 1.27)
+			)
+			(justify left bottom)
+		)
+	)
 	(label "ESPJTAG.TDI"
 		(at 30.48 167.64 0)
@@
 	(label "ESPJTAG.TDO"
 		(at 162.56 146.05 0)
+		(effects
+			(font
+				(size 1.27 1.27)
+			)
+			(justify left bottom)
+		)
+	)
+	(label "unconnected-(U40-NC-Pad28)"
+		(at 149.86 133.35 0)
 		(effects
 			(font
@@
 		(dnp no)
 		(fields_autoplaced yes)
-		(property "Reference" "R110"
+		(property "Reference" "R105"
 			(at 173.99 149.8599 0)
 			(show_name no)
@@
 			(project "tonnere"
 				(path "/eb8e239c-f2ec-4b57-8f5c-6c75d6b59ab3/46474bdc-762b-418e-b7cb-754958627956"
-					(reference "R110")
+					(reference "R105")
 					(unit 1)
 				)
@@
 		(dnp no)
 		(fields_autoplaced yes)
-		(property "Reference" "R103"
+		(property "Reference" "R98"
 			(at 34.29 138.4299 0)
 			(show_name no)
@@
 			(project "tonnere"
 				(path "/eb8e239c-f2ec-4b57-8f5c-6c75d6b59ab3/46474bdc-762b-418e-b7cb-754958627956"
-					(reference "R103")
+					(reference "R98")
 					(unit 1)
 				)
@@
 		(dnp no)
 		(fields_autoplaced yes)
-		(property "Reference" "R121"
+		(property "Reference" "R116"
 			(at 114.3 91.4399 0)
 			(show_name no)
@@
 			(project "tonnere"
 				(path "/eb8e239c-f2ec-4b57-8f5c-6c75d6b59ab3/46474bdc-762b-418e-b7cb-754958627956"
-					(reference "R121")
+					(reference "R116")
 					(unit 1)
 				)
@@
 		(dnp no)
 		(fields_autoplaced yes)
-		(property "Reference" "R108"
+		(property "Reference" "R103"
 			(at 36.83 172.7199 0)
 			(show_name no)
@@
 			(project "tonnere"
 				(path "/eb8e239c-f2ec-4b57-8f5c-6c75d6b59ab3/46474bdc-762b-418e-b7cb-754958627956"
-					(reference "R108")
+					(reference "R103")
 					(unit 1)
 				)
@@
 		(dnp no)
 		(fields_autoplaced yes)
-		(property "Reference" "R106"
+		(property "Reference" "R101"
 			(at 194.31 91.4399 0)
 			(show_name no)
@@
 			(project "tonnere"
 				(path "/eb8e239c-f2ec-4b57-8f5c-6c75d6b59ab3/46474bdc-762b-418e-b7cb-754958627956"
-					(reference "R106")
+					(reference "R101")
 					(unit 1)
 				)
@@
 		(dnp no)
 		(fields_autoplaced yes)
-		(property "Reference" "C117"
+		(property "Reference" "C118"
 			(at 267.97 67.3099 0)
 			(show_name no)
@@
 			(project "tonnere"
 				(path "/eb8e239c-f2ec-4b57-8f5c-6c75d6b59ab3/46474bdc-762b-418e-b7cb-754958627956"
-					(reference "C117")
+					(reference "C118")
 					(unit 1)
 				)
@@
 		(dnp no)
 		(fields_autoplaced yes)
-		(property "Reference" "J23"
+		(property "Reference" "J22"
 			(at 50.8 151.13 0)
 			(show_name no)
@@
 			(project "tonnere"
 				(path "/eb8e239c-f2ec-4b57-8f5c-6c75d6b59ab3/46474bdc-762b-418e-b7cb-754958627956"
-					(reference "J23")
+					(reference "J22")
 					(unit 1)
 				)
@@
 		(dnp no)
 		(fields_autoplaced yes)
-		(property "Reference" "J19"
+		(property "Reference" "J18"
 			(at 228.6 68.5799 0)
 			(show_name no)
@@
 			(project "tonnere"
 				(path "/eb8e239c-f2ec-4b57-8f5c-6c75d6b59ab3/46474bdc-762b-418e-b7cb-754958627956"
-					(reference "J19")
+					(reference "J18")
 					(unit 1)
 				)
@@
 		(in_pos_files yes)
 		(dnp no)
-		(property "Reference" "C115"
+		(property "Reference" "C116"
 			(at 255.27 67.3099 0)
 			(show_name no)
@@
 			(project "tonnere"
 				(path "/eb8e239c-f2ec-4b57-8f5c-6c75d6b59ab3/46474bdc-762b-418e-b7cb-754958627956"
-					(reference "C115")
+					(reference "C116")
 					(unit 1)
 				)
@@
 		(dnp no)
 		(fields_autoplaced yes)
-		(property "Reference" "R113"
+		(property "Reference" "R108"
 			(at 177.8 90.1699 0)
 			(show_name no)
@@
 			(project "tonnere"
 				(path "/eb8e239c-f2ec-4b57-8f5c-6c75d6b59ab3/46474bdc-762b-418e-b7cb-754958627956"
-					(reference "R113")
+					(reference "R108")
 					(unit 1)
 				)
@@
 		(dnp no)
 		(fields_autoplaced yes)
-		(property "Reference" "U40"
+		(property "Reference" "U41"
 			(at 134.62 97.79 0)
 			(show_name no)
@@
 			(project "tonnere"
 				(path "/eb8e239c-f2ec-4b57-8f5c-6c75d6b59ab3/46474bdc-762b-418e-b7cb-754958627956"
-					(reference "U40")
+					(reference "U41")
 					(unit 1)
 				)
