File: board/kicad/tonnere/io_cards.kicad_sch (KiCad schematic)
At the start: 11 parts, among them U46 TPD4E02B04DQA, U47 TPD4E02B04DQA

Commit message: Changed video dac to 5 bit R2R and 6th-8th bits as pattern and/or sigma delta.
Parts:
- renumbered C122 to C123, C123 to C124, C53 to C56, C54 to C57, RN12 to RN20, RN13 to RN21, U46 to U47, U47 to U48
Connections:
- net unconnected-(U47-NC-Pad10): now reaches U48.10 (NC)
- net unconnected-(U47-NC-Pad6): now reaches U48.6 (NC)
- net unconnected-(U47-NC-Pad7): now reaches U48.7 (NC)
- net unconnected-(U47-NC-Pad9): now reaches U48.9 (NC)
- net unconnected-(U46-NC-Pad10): now reaches U47.10 (NC)
- net unconnected-(U46-NC-Pad6): now reaches U47.6 (NC)
- net unconnected-(U46-NC-Pad7): now reaches U47.7 (NC)
- net unconnected-(U46-NC-Pad9): now reaches U47.9 (NC)
- net unconnected-(RN12-R1.2-Pad8): now reaches RN20.8 (R1.2)
Changed lines of the file:
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@@
+		)
+	)
+	(label "unconnected-(U47-NC-Pad7)"
+		(at 153.67 77.47 90)
+		(effects
+			(font
+				(size 1.27 1.27)
+			)
+			(justify left bottom)
 		)
 	)
@@
 		)
 	)
+	(label "unconnected-(U46-NC-Pad9)"
+		(at 123.19 77.47 90)
+		(effects
+			(font
+				(size 1.27 1.27)
+			)
+			(justify left bottom)
+		)
+	)
 	(label "SD.WP"
 		(at 158.75 34.29 0)
@@
 		)
 	)
+	(label "unconnected-(U46-NC-Pad6)"
+		(at 110.49 77.47 90)
+		(effects
+			(font
+				(size 1.27 1.27)
+			)
+			(justify left bottom)
+		)
+	)
+	(label "unconnected-(RN12-R1.2-Pad8)"
+		(at 114.3 27.94 270)
+		(effects
+			(font
+				(size 1.27 1.27)
+			)
+			(justify right bottom)
+		)
+	)
 	(label "SD.D1"
 		(at 102.87 34.29 0)
@@
 		)
 	)
+	(label "unconnected-(U47-NC-Pad9)"
+		(at 161.29 77.47 90)
+		(effects
+			(font
+				(size 1.27 1.27)
+			)
+			(justify left bottom)
+		)
+	)
+	(label "unconnected-(U46-NC-Pad7)"
+		(at 115.57 77.47 90)
+		(effects
+			(font
+				(size 1.27 1.27)
+			)
+			(justify left bottom)
+		)
+	)
+	(label "unconnected-(U46-NC-Pad10)"
+		(at 128.27 77.47 90)
+		(effects
+			(font
+				(size 1.27 1.27)
+			)
+			(justify left bottom)
+		)
+	)
+	(label "unconnected-(U47-NC-Pad6)"
+		(at 148.59 77.47 90)
+		(effects
+			(font
+				(size 1.27 1.27)
+			)
+			(justify left bottom)
+		)
+	)
 	(label "SD.D3"
 		(at 102.87 39.37 0)
@@
 	(label "SD.DETECT"
 		(at 158.75 31.75 0)
+		(effects
+			(font
+				(size 1.27 1.27)
+			)
+			(justify left bottom)
+		)
+	)
+	(label "unconnected-(U47-NC-Pad10)"
+		(at 166.37 77.47 90)
 		(effects
 			(font
@@
 		(in_pos_files yes)
 		(dnp no)
-		(property "Reference" "U47"
+		(property "Reference" "U48"
 			(at 172.72 83.8199 90)
 			(show_name no)
@@
 			(project "tonnere"
 				(path "/eb8e239c-f2ec-4b57-8f5c-6c75d6b59ab3/6e470164-ad0d-4d1f-a1f3-2d1a639770a2"
-					(reference "U47")
+					(reference "U48")
 					(unit 1)
 				)
@@
 		(in_pos_files yes)
 		(dnp no)
-		(property "Reference" "U46"
+		(property "Reference" "U47"
 			(at 134.62 83.8199 90)
 			(show_name no)
@@
 			(project "tonnere"
 				(path "/eb8e239c-f2ec-4b57-8f5c-6c75d6b59ab3/6e470164-ad0d-4d1f-a1f3-2d1a639770a2"
-					(reference "U46")
+					(reference "U47")
 					(unit 1)
 				)
@@
 		(dnp no)
 		(fields_autoplaced yes)
-		(property "Reference" "RN13"
+		(property "Reference" "RN21"
 			(at 163.83 20.3199 0)
 			(show_name no)
@@
 			(project "tonnere"
 				(path "/eb8e239c-f2ec-4b57-8f5c-6c75d6b59ab3/6e470164-ad0d-4d1f-a1f3-2d1a639770a2"
-					(reference "RN13")
+					(reference "RN21")
 					(unit 1)
 				)
@@
 		(dnp no)
 		(fields_autoplaced yes)
-		(property "Reference" "C54"
+		(property "Reference" "C57"
 			(at 217.17 35.5599 0)
 			(show_name no)
@@
 			(project "tonnere"
 				(path "/eb8e239c-f2ec-4b57-8f5c-6c75d6b59ab3/6e470164-ad0d-4d1f-a1f3-2d1a639770a2"
-					(reference "C54")
+					(reference "C57")
 					(unit 1)
 				)
@@
 		(dnp no)
 		(fields_autoplaced yes)
-		(property "Reference" "C122"
+		(property "Reference" "C123"
 			(at 201.93 35.5599 0)
 			(show_name no)
@@
 			(project "tonnere"
 				(path "/eb8e239c-f2ec-4b57-8f5c-6c75d6b59ab3/6e470164-ad0d-4d1f-a1f3-2d1a639770a2"
-					(reference "C122")
+					(reference "C123")
 					(unit 1)
 				)
@@
 		(dnp no)
 		(fields_autoplaced yes)
-		(property "Reference" "C123"
+		(property "Reference" "C124"
 			(at 246.38 35.5599 0)
 			(show_name no)
@@
 			(project "tonnere"
 				(path "/eb8e239c-f2ec-4b57-8f5c-6c75d6b59ab3/6e470164-ad0d-4d1f-a1f3-2d1a639770a2"
-					(reference "C123")
+					(reference "C124")
 					(unit 1)
 				)
@@
 		(dnp no)
 		(fields_autoplaced yes)
-		(property "Reference" "C53"
+		(property "Reference" "C56"
 			(at 232.41 35.5599 0)
 			(show_name no)
@@
 			(project "tonnere"
 				(path "/eb8e239c-f2ec-4b57-8f5c-6c75d6b59ab3/6e470164-ad0d-4d1f-a1f3-2d1a639770a2"
-					(reference "C53")
+					(reference "C56")
 					(unit 1)
 				)
@@
 		(dnp no)
 		(fields_autoplaced yes)
-		(property "Reference" "RN12"
+		(property "Reference" "RN20"
 			(at 116.84 21.5899 0)
 			(show_name no)
@@
 			(project "tonnere"
 				(path "/eb8e239c-f2ec-4b57-8f5c-6c75d6b59ab3/6e470164-ad0d-4d1f-a1f3-2d1a639770a2"
-					(reference "RN12")
+					(reference "RN20")
 					(unit 1)
 				)
