File: board/kicad/tonnere/ram.kicad_sch (KiCad schematic)
At the start: 8 parts, among them U31 IS61WV204816BLL-10BLI, U36 IS61WV204816BLL-10BLI, U42 AS4C16M16SA

Commit message: Changed video dac to 5 bit R2R and 6th-8th bits as pattern and/or sigma delta.
Parts:
- renumbered C108 to C109, C109 to C110, C94 to C95, R112 to R107, U31 to U32, U36 to U37, U42 to U43
Connections:
- net Net-(U42-CLK): now reaches R107.2, U43.38 (CLK)
- net unconnected-(U42-NC/RFU-Pad40): now reaches U43.40 (NC/RFU)
- net unconnected-(U36-NC-PadA6): now reaches U37.A6 (NC)
- net unconnected-(U36-NC-PadE3): now reaches U37.E3 (NC)
- net unconnected-(U31-NC-PadA6): now reaches U32.A6 (NC)
- net unconnected-(U31-NC-PadE3): now reaches U32.E3 (NC)
Changed lines of the file:
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@@
+		)
+	)
+	(label "unconnected-(U42-NC{slash}RFU-Pad40)"
+		(at 121.92 247.65 0)
+		(effects
+			(font
+				(size 1.27 1.27)
+			)
+			(justify left bottom)
 		)
 	)
@@
 		)
 	)
+	(label "unconnected-(U36-NC-PadE3)"
+		(at 341.63 194.31 0)
+		(effects
+			(font
+				(size 1.27 1.27)
+			)
+			(justify left bottom)
+		)
+	)
 	(label "SRAM2.A20"
 		(at 345.44 140.97 0)
@@
 		)
 	)
+	(label "unconnected-(U31-NC-PadE3)"
+		(at 134.62 104.14 0)
+		(effects
+			(font
+				(size 1.27 1.27)
+			)
+			(justify left bottom)
+		)
+	)
 	(label "SRAM1.CE_N"
 		(at 73.66 76.2 0)
@@
 		)
 	)
+	(label "unconnected-(U31-NC-PadA6)"
+		(at 88.9 63.5 180)
+		(effects
+			(font
+				(size 1.27 1.27)
+			)
+			(justify right bottom)
+		)
+	)
 	(label "SRAM1.D3"
 		(at 73.66 106.68 0)
@@
 		)
 	)
+	(label "Net-(U42-CLK)"
+		(at 99.06 245.11 180)
+		(effects
+			(font
+				(size 1.27 1.27)
+			)
+			(justify right bottom)
+		)
+	)
 	(label "SRAM2.D14"
 		(at 345.44 184.15 0)
@@
 		)
 	)
+	(label "Net-(U42-CLK)"
+		(at 99.06 245.11 180)
+		(effects
+			(font
+				(size 1.27 1.27)
+			)
+			(justify right bottom)
+		)
+	)
 	(label "SDRAM1.DQ14"
 		(at 132.08 232.41 0)
@@
 			)
 			(justify left bottom)
+		)
+	)
+	(label "unconnected-(U36-NC-PadA6)"
+		(at 295.91 153.67 180)
+		(effects
+			(font
+				(size 1.27 1.27)
+			)
+			(justify right bottom)
 		)
 	)
@@
 		(dnp no)
 		(fields_autoplaced yes)
-		(property "Reference" "C109"
+		(property "Reference" "C110"
 			(at 359.41 43.1799 0)
 			(show_name no)
@@
 			(project "tonnere"
 				(path "/eb8e239c-f2ec-4b57-8f5c-6c75d6b59ab3/697ece47-2a2f-49f7-b3cd-8d11bcc6cfcf"
-					(reference "C109")
+					(reference "C110")
 					(unit 1)
 				)
@@
 		(dnp no)
 		(fields_autoplaced yes)
-		(property "Reference" "U42"
+		(property "Reference" "U43"
 			(at 113.9033 189.23 0)
 			(show_name no)
@@
 			(project "tonnere"
 				(path "/eb8e239c-f2ec-4b57-8f5c-6c75d6b59ab3/697ece47-2a2f-49f7-b3cd-8d11bcc6cfcf"
-					(reference "U42")
+					(reference "U43")
 					(unit 1)
 				)
@@
 		(dnp no)
 		(fields_autoplaced yes)
-		(property "Reference" "C108"
+		(property "Reference" "C109"
 			(at 349.25 43.1799 0)
 			(show_name no)
@@
 			(project "tonnere"
 				(path "/eb8e239c-f2ec-4b57-8f5c-6c75d6b59ab3/697ece47-2a2f-49f7-b3cd-8d11bcc6cfcf"
-					(reference "C108")
+					(reference "C109")
 					(unit 1)
 				)
@@
 		(in_pos_files yes)
 		(dnp no)
-		(property "Reference" "R112"
+		(property "Reference" "R107"
 			(at 97.282 243.84 90)
 			(show_name no)
@@
 			(project "tonnere"
 				(path "/eb8e239c-f2ec-4b57-8f5c-6c75d6b59ab3/697ece47-2a2f-49f7-b3cd-8d11bcc6cfcf"
-					(reference "R112")
+					(reference "R107")
 					(unit 1)
 				)
@@
 		(dnp no)
 		(fields_autoplaced yes)
-		(property "Reference" "C94"
+		(property "Reference" "C95"
 			(at 337.82 43.1799 0)
 			(show_name no)
@@
 			(project "tonnere"
 				(path "/eb8e239c-f2ec-4b57-8f5c-6c75d6b59ab3/697ece47-2a2f-49f7-b3cd-8d11bcc6cfcf"
-					(reference "C94")
+					(reference "C95")
 					(unit 1)
 				)
@@
 		(dnp no)
 		(fields_autoplaced yes)
-		(property "Reference" "U36"
+		(property "Reference" "U37"
 			(at 318.77 130.81 0)
 			(show_name no)
@@
 			(project "tonnere"
 				(path "/eb8e239c-f2ec-4b57-8f5c-6c75d6b59ab3/697ece47-2a2f-49f7-b3cd-8d11bcc6cfcf"
-					(reference "U36")
+					(reference "U37")
 					(unit 1)
 				)
@@
 		(dnp no)
 		(fields_autoplaced yes)
-		(property "Reference" "U31"
+		(property "Reference" "U32"
 			(at 111.76 40.64 0)
 			(show_name no)
@@
 			(project "tonnere"
 				(path "/eb8e239c-f2ec-4b57-8f5c-6c75d6b59ab3/697ece47-2a2f-49f7-b3cd-8d11bcc6cfcf"
-					(reference "U31")
+					(reference "U32")
 					(unit 1)
 				)
