File: board/kicad/tonnere/usb.kicad_sch (KiCad schematic)
At the start: 51 parts, among them J20 USB_A, J21 73725-1180RLF, J25 73725-1180RLF, J26 73725-1180RLF, U34 AP2553AW6-7, U38 AP2553AW6-7, U39 AP2553AW6-7, U41 AP2553AW6-7, U43 TPD4E02B04DQA, U44 USB2514B_Bi, U45 TPD4E02B04DQA, Y9 24MHz

Commit message: Changed video dac to 5 bit R2R and 6th-8th bits as pattern and/or sigma delta.
Parts:
- renumbered C100 to C101, C104 to C105, C105 to C106, C106 to C107, C107 to C108, C110 to C111, C111 to C112, C112 to C113, C114 to C115, C118 to C119, C119 to C120, C120 to C121, C121 to C122, C124 to C125, C125 to C126, C82 to C83, C87 to C88, C89 to C90, C93 to C94, C95 to C96, C98 to C99, FB6 to FB5, J20 to J19, J21 to J20, J25 to J24, J26 to J25, R105 to R100, R107 to R102, R109 to R104, R111 to R106, R114 to R109, R117 to R112, R119 to R114, R122 to R117, R124 to R119, R125 to R120, R127 to R122, R128 to R123, R132 to R127, R133 to R128, U34 to U35, U38 to U39, U39 to U40, U41 to U42, U43 to U44, U44 to U45, U45 to U46
Connections:
- net Net-(U34-FAULT#): now reaches R102.2, U35.4 (FAULT#), U45.21 (OCS_N4)
- net Net-(U39-ILIM): now reaches R109.1, U40.5 (ILIM)
- net Net-(U44-HS_IND/CFG_SEL1): now reaches R122.2, U45.25 (HS_IND/CFG_SEL1)
- net Net-(U44-SCL/SMBCLK/CFG_SEL0): now reaches R120.2, U45.24 (SCL/SMBCLK/CFG_SEL0)
- net Net-(U44-SDA/SMBDATA/NON_REM1): now reaches R119.2, U45.22 (SDA/SMBDATA/NON_REM1)
- net Net-(J20-D-): now reaches J19.2 (D-), U44.2 (IO2), U45.8 (USBDM_DN4/PRT_DIS_M4)
- net Net-(J20-D+): now reaches J19.3 (D+), U44.1 (IO1), U45.9 (USBDP_DN4/PRT_DIS_P4)
- net Net-(U41-FAULT#): now reaches R117.2, U42.4 (FAULT#), U45.13 (OCS_N1)
- net Net-(U39-EN/EN#): now reaches U40.3 (EN/EN#), U45.16 (PRTPWR2/BC_EN2)
- net Net-(U39-FAULT#): now reaches R112.2, U40.4 (FAULT#), U45.17 (OCS_N2)
- net unconnected-(U43-NC-Pad10): now reaches U44.10 (NC)
- net Net-(J21-D+): now reaches J20.3 (D+), U44.4 (IO3), U45.7 (USBDP_DN3/PRT_DIS_P3)
- net Net-(J21-D-): now reaches J20.2 (D-), U44.5 (IO4), U45.6 (USBDM_DN3/PRT_DIS_M3)
- net unconnected-(U43-NC-Pad6): now reaches U44.6 (NC)
- net unconnected-(U43-NC-Pad7): now reaches U44.7 (NC)
- net unconnected-(U43-NC-Pad9): now reaches U44.9 (NC)
- net Net-(U44-XTALOUT): now reaches C126.2, U45.32 (XTALOUT), Y9.1
- net Net-(J25-D+): now reaches J24.3 (D+), U45.4 (USBDP_DN2/PRT_DIS_P2), U46.1 (IO1)
- net unconnected-(U45-NC-Pad10): now reaches U46.10 (NC)
- net Net-(J25-D-): now reaches J24.2 (D-), U45.3 (USBDM_DN2/PRT_DIS_M2), U46.2 (IO2)
- net Net-(J26-D+): now reaches J25.3 (D+), U45.2 (USBDP_DN1/PRT_DIS_P1), U46.4 (IO3)
- net Net-(J26-D-): now reaches J25.2 (D-), U45.1 (USBDM_DN1/PRT_DIS_M1), U46.5 (IO4)
- net unconnected-(U45-NC-Pad6): now reaches U46.6 (NC)
- net unconnected-(U45-NC-Pad7): now reaches U46.7 (NC)
- net unconnected-(U45-NC-Pad9): now reaches U46.9 (NC)
- net Net-(U34-EN/EN#): now reaches U35.3 (EN/EN#), U45.20 (PRTPWR4/BC_EN4)
- net Net-(U34-ILIM): now reaches R100.1, U35.5 (ILIM)
- net Net-(U44-SUSP_IND/LOCAL_PWR/NON_REM0): now reaches R127.2, U45.28 (SUSP_IND/LOCAL_PWR/NON_REM0)
- net Net-(U44-RESET_N): now reaches R123.2, U45.26 (RESET_N)
- net Net-(U38-ILIM): now reaches R104.1, U39.5 (ILIM)
- net Net-(U44-XTALIN/CLKIN): now reaches C125.2, U45.33 (XTALIN/CLKIN), Y9.3
- net Net-(U38-EN/EN#): now reaches U39.3 (EN/EN#), U45.18 (PRTPWR3/BC_EN3)
- net Net-(U38-FAULT#): now reaches R106.2, U39.4 (FAULT#), U45.19 (OCS_N3)
- net Net-(U44-CRFILT): now reaches C112.2, U45.14 (CRFILT)
- net Net-(U41-EN/EN#): now reaches U42.3 (EN/EN#), U45.12 (PRTPWR1/BC_EN1)
- net Net-(U41-ILIM): now reaches R114.1, U42.5 (ILIM)
- net unconnected-(U44-TEST-Pad11): now reaches U45.11 (TEST)
- net Net-(U44-PLLFILT): now reaches C122.2, U45.34 (PLLFILT)
- net Net-(U44-RBIAS): now reaches R128.2, U45.35 (RBIAS)
